Commit message: Set new colors to wheels

File: ca_description/urdf/create_base_gazebo.urdf.xacro (robot description, xacro)
@@ -64,4 +64,5 @@
       <minDepth>0.001</minDepth>
       <maxVel>1.0</maxVel>
+      <material>Gazebo/Grey</material>
     </gazebo>
     <gazebo reference="right_wheel_link">
@@ -72,4 +73,5 @@
       <minDepth>0.001</minDepth>
       <maxVel>1.0</maxVel>
+      <material>Gazebo/Grey</material>
     </gazebo>
   </xacro:macro>

File: ca_description/urdf/create_caster_wheel.xacro (robot description, xacro)
@@ -34,4 +34,7 @@
     <axis xyz="0 1 0" />
   </joint>
+  <gazebo reference="${link_name}">
+    <material>Gazebo/Grey</material>
+  </gazebo>
 </xacro:macro>
 </robot>
